File: pcb_r/pcb_r.kicad_pcb (KiCad board)
At the start: 2 copper layers, 133.4 x 104.8 mm, 47 parts, among them J1 MJ-4PP-9, SW23 SW_PUSH, SW24 SW_PUSH, SW25 SW_PUSH, SW26 SW_PUSH, SW27 SW_PUSH, SW28 SW_PUSH, SW29 SW_PUSH, SW30 SW_PUSH, SW31 SW_PUSH, SW32 SW_PUSH, SW33 SW_PUSH, SW34 SW_PUSH, SW35 SW_PUSH, SW36 SW_PUSH, SW37 SW_PUSH, SW38 SW_PUSH, SW39 SW_PUSH, SW40 SW_PUSH, SW41 SW_PUSH, SW42 SW_PUSH, SW43 SW_PUSH, SW44 SW_PUSH, U1 ProMicro

Commit message: added gnd mask
Parts:
- added Ref**: Val**, kbd:spacer_m2, F.Cu at (171.4, 59.5)
- added Ref**: Val**, kbd:spacer_m2, F.Cu at (261.9, 59.5)
- added Ref**: Val**, kbd:spacer_m2, F.Cu at (223.8, 45.2)
- added Ref**: Val**, kbd:spacer_m2, F.Cu at (261.9, 40.5)
- added Ref**: Val**, kbd:spacer_m2, F.Cu at (171.4, 108.3)
- added Ref**: Val**, kbd:spacer_m2, F.Cu at (223.8, 83.3)
Routing:
- net COL4: track 142.9 -> 146.2 mm
- net COL3: track 126.2 -> 123.0 mm, vias 7 -> 6
- net COL5: track 132.0 -> 134.0 mm
- net ROW4: track 124.3 -> 125.8 mm, vias 2 -> 3
- net COL1: track 89.9 -> 91.0 mm
- added copper zone on B.Cu, net GND
- added copper zone on F.Cu, net GND
Other:
- board text added: "Maggie44 by Tamaroh Ver 1.0"

Commit message: fixed #4
Routing:
- net COL3: track 123.0 -> 142.1 mm, vias 6 -> 8
Changed lines of the file:
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@@
   (segment (start 207.16875 73.81875) (end 207.16875 89.296875) (width 0.25) (layer "F.Cu") (net 34))
   (segment (start 207.16875 54.76875) (end 207.16875 69.05625) (width 0.25) (layer "F.Cu") (net 34))
+  (segment (start 207.16875 35.71875) (end 207.16875 50.00625) (width 0.25) (layer "F.Cu") (net 34))
   (via (at 207.16875 54.76875) (size 0.8) (drill 0.4) (layers "F.Cu" "B.Cu") (net 34))
   (via (at 207.16875 73.81875) (size 0.8) (drill 0.4) (layers "F.Cu" "B.Cu") (net 34))
@@
   (via (at 162.9624 63.103125) (size 0.8) (drill 0.4) (layers "F.Cu" "B.Cu") (net 34))
   (via (at 162.9624 78.58125) (size 0.8) (drill 0.4) (layers "F.Cu" "B.Cu") (net 34))
+  (via (at 207.16875 50.00625) (size 0.8) (drill 0.4) (layers "F.Cu" "B.Cu") (net 34))
+  (via (at 207.16875 35.71875) (size 0.8) (drill 0.4) (layers "F.Cu" "B.Cu") (net 34))
   (segment (start 192.94 91.736875) (end 192.94 95.09125) (width 0.25) (layer "B.Cu") (net 34))
+  (segment (start 207.16875 52.17) (end 207.2275 52.22875) (width 0.25) (layer "B.Cu") (net 34))
   (segment (start 205.978125 90.4875) (end 194.071875 90.4875) (width 0.25) (layer "B.Cu") (net 34))
   (segment (start 207.2275 52.22875) (end 207.2275 54.71) (width 0.25) (layer "B.Cu") (net 34))
   (segment (start 182.330945 78.58125) (end 185.7375 75.174695) (width 0.25) (layer "B.Cu") (net 34))
   (segment (start 163.391025 62.6745) (end 162.9624 63.103125) (width 0.25) (layer "B.Cu") (net 34))
+  (segment (start 207.2275 35.66) (end 207.16875 35.71875) (width 0.25) (layer "B.Cu") (net 34))
+  (segment (start 207.16875 50.00625) (end 207.16875 52.17) (width 0.25) (layer "B.Cu") (net 34))
   (segment (start 162.9624 78.58125) (end 182.330945 78.58125) (width 0.25) (layer "B.Cu") (net 34))
   (segment (start 207.2275 54.71) (end 207.16875 54.76875) (width 0.25) (layer "B.Cu") (net 34))
@@
   (segment (start 207.16875 69.05625) (end 207.16875 71.22) (width 0.25) (layer "B.Cu") (net 34))
   (segment (start 189.309375 69.05625) (end 207.16875 69.05625) (width 0.25) (layer "B.Cu") (net 34))
+  (segment (start 207.2275 33.17875) (end 207.2275 35.66) (width 0.25) (layer "B.Cu") (net 34))
   (segment (start 164.7739 62.6745) (end 163.391025 62.6745) (width 0.25) (layer "B.Cu") (net 34))
   (segment (start 192.88125 91.678125) (end 192.94 91.736875) (width 0.25) (layer "B.Cu") (net 34))
